Commit message: gazebo pluigins added

File: urdf/my_robot_gazebo.xacro (robot description, xacro)
@@ -1,3 +1,58 @@
 <?xml version ="1.0"?>
-<robot xmlns:zacro="http://www.ros.org/wiki/xacro" name="my_robot">
+<robot xmlns:xacro="http://www.ros.org/wiki/xacro" name="my_robot">
+    <transmission name="right_wheel_transmission">
+        <plugin>transmission_interface/SimpleTransmission</plugin>
+        <actuator name="right_wheel_motor" role = "actuator_right"/>
+        <joint name="base_wheel_right_joint" role = "joint_right">
+            <mechanicalReduction>1.0</mechanicalReduction>
+        </joint>
+    </transmission>
+    <transmission name="left_wheel_transmission">
+        <plugin>transmission_interface/SimpleTransmission</plugin>
+        <actuator name="left_wheel_motor" role = "actuator_left"/>
+        <joint name="base_wheel_left_joint" role = "joint_left">
+            <mechanicalReduction>1.0</mechanicalReduction>
+        </joint>
+    </transmission>
+    <gazebo reference = "right_wheel_link">
+        <mu1>100000000000000.0</mu1><!--(coef of friction)it is set to extremly haigh number to avoid any slipping-->
+        <mu2>100000000000000.0</mu2><!--it is set to extremly haigh number to avoid any slipping-->
+        <kp>1000000000000.0</kp><!--gazebo plugin-->
+        <kd>10.0</kd>
+        <minDepth>0.001</minDepth><!--solver accuracy-->
+        <maxVel>0.1</maxVel>
+        <fdir1>1 0 0</fdir1>
+    </gazebo>
+    <gazebo reference = "left_wheel_link">
+        <mu1>100000000000000.0</mu1><!--(coef of friction)it is set to extremly haigh number to avoid any slipping-->
+        <mu2>100000000000000.0</mu2><!--it is set to extremly haigh number to avoid any slipping-->
+        <kp>1000000000000.0</kp><!--gazebo plugin-->
+        <kd>10.0</kd>
+        <minDepth>0.001</minDepth><!--solver accuracy-->
+        <maxVel>0.1</maxVel>
+        <fdir1>1 0 0</fdir1>
+    </gazebo>
+    <gazebo reference = "caster_wheel_rear">
+        <mu1>0.1</mu1><!--(coef of friction)it is set to extremly haigh number to avoid any slipping-->
+        <mu2>0.1</mu2><!--it is set to extremly haigh number to avoid any slipping-->
+        <kp>1000000.0</kp><!--gazebo plugin-->
+        <kd>100.0</kd>
+        <minDepth>0.001</minDepth><!--solver accuracy-->
+        <maxVel>0.1</maxVel>
+    </gazebo>
+    <gazebo reference = "caster_wheel_front">
+        <mu1>0.1</mu1><!--(coef of friction)it is set to extremly haigh number to avoid any slipping-->
+        <mu2>0.1</mu2><!--it is set to extremly haigh number to avoid any slipping-->
+        <kp>1000000.0</kp><!--gazebo plugin-->
+        <kd>100.0</kd>
+        <minDepth>0.001</minDepth><!--solver accuracy-->
+        <maxVel>0.1</maxVel>
+    </gazebo>
+    <gazebo>
+        <plugin filename="libgazebo_ros2_control.so" name="gazebo_ros2_control">
+            <robot_param>robot_description</robot_param>
+            <robot_param_node>robot_state_publisher</robot_param_node>
+            <parameters></parameters>
+        </plugin>
+    </gazebo>
 </robot>

File: urdf/robot_urdf.xacro (robot description, xacro)
@@ -1,8 +1,16 @@
 <?xml version ="1.0"?>
-<robot xmlns:zacro="http://www.ros.org/wiki/xacro" name="my_robot">
-   <xacro:include filename="xacroFile"/>
+<robot xmlns:xacro="http://www.ros.org/wiki/xacro" name="my_robot">
+    <xacro:include filename="$(find my_robot_description)/urdf/my_robot_gazebo.xacro"/>
+<xacro:include filename="$(find my_robot_description)/urdf/urdf/urdf/my_robot_ros2_control.xacro"/>
     <link name="base_fooprint"/>
              <!-- footprint usualy the lower part of the robot touched to the ground at point 0 0 0 -->
-    <link name=" ">
+    <link name="base_link">
+        <inertial>
+            <origin xyz="0 0 0.04" rpy="0.0 0.25 0.3" />
+            <mass value="8.2573504e-01"/>
+            <inertia ixx="2.2124416e-02" ixy="-1.2294101e-04" ixz="3.4938785e-04"
+                    iyy="2.1193702e-02" iyz="-5.0120904e-05"
+                    izz="2.0064271e-02" />
+        </inertial>
         <visual>
             <origin rpy="0 0 0" xyz="0 0 0" />
@@ -12,12 +20,13 @@
                </geometry>
                <material name="blue">
-                    <color rgba="0.0 0.0 1.0 1.0"/> <!-- RGB and Alpha values (1.0 = fully opaque) -->
+                    <color rgba="0.0 0.0 1.0 1.0"/>
+                    <!-- RGB and Alpha values (1.0 = fully opaque) -->
                </material>
                <collision>
-                <origin rpy="0 0 0" xyz="0 0 0" />
-                <geometry>
-                    <mesh filename="package://my_robot_description/meshes/base_link.STL" />
-                </geometry>
-            </collision>
+                    <origin rpy="0 0 0" xyz="0 0 0" />
+                    <geometry>
+                        <mesh filename="package://my_robot_description/meshes/base_link.STL" />
+                    </geometry>
+                </collision>
         </visual>
     </link>
@@ -30,4 +39,11 @@
     </joint>
     <link name="caster_wheel_front">
+            <inertial>
+            <origin xyz="3.89968128948481E-07 2.40073004698083E-07 0.00219173397061506" rpy="0 0 0" />
+            <mass value="1.44379265037903E-06" />
+            <inertia ixx="7.23075276010246E-11" ixy="-6.10956883467859E-16" ixz="2.22849693525031E-15"
+                    iyy="3.8713793085917E-11"  iyz="2.93909858781952E-15"
+                    izz="1.00967486676306E-10" />
+            </inertial>
             <visual>
                 <origin rpy="0 0 0" xyz="0 0 0" />
@@ -39,4 +55,10 @@
                 </material>
             </visual>
+            <collision>
+                <origin xyz="0.0 0.0 0.0" rpy="0.0 0.0 0.0"/>
+                <geometry>
+                     <sphere radius="0.005"/>
+                </geometry>
+            </collision>
     </link>
     <joint name="base_caster_wheel_front_joint" type="fixed">
@@ -46,4 +68,11 @@
     </joint>
    <link name="caster_wheel_rear">
+            <inertial>
+            <origin xyz="3.8996812895542E-07 2.40073004698083E-07 0.00219173397061509" rpy="0 0 0" />
+            <mass value="1.44379265037902E-06" />
+            <inertia ixx="7.23075276010246E-11" ixy="-6.10956872363424E-16" ixz="2.22849693527207E-15"
+                    iyy="3.87137930859167E-11" iyz="2.939098587861E-15"
+                    izz="1.00967486676306E-10" />
+            </inertial>
             <visual>
                 <origin rpy="0 0 0" xyz="0 0 0" />
@@ -55,4 +84,10 @@
                 </material>
             </visual>
+            <collision>
+                <origin xyz="0.0 0.0 0.0" rpy="0.0 0.0 0.0"/>
+                <geometry>
+                        <sphere radius="0.005"/>
+                </geometry>
+            </collision>
     </link>
     <joint name="base_caster_wheel_rear_joint" type="fixed">
@@ -62,4 +97,11 @@
     </joint>
     <link name="right_wheel_link">
+            <inertial>
+            <origin xyz="0 -0.014 0" rpy="0 0 0" />
+            <mass value="0.0530086090966721" />
+            <inertia ixx="1.88176298336665E-05" ixy="-4.8444933029987E-10" ixz="1.88163708851143E-08"
+                    iyy="3.11510738647764E-05" iyz="-6.93560663069607E-11"
+                    izz="1.8801969558182E-05" />
+            </inertial>
             <visual>
                 <origin rpy="1.57 0 0" xyz="0 0 0" />
@@ -86,4 +128,11 @@
     </joint>
  <link name="left_wheel_link">
+           <inertial>
+                <origin xyz="0 0.014 0" rpy="0 0 0" />
+                <mass value="0.0530086043217644" />
+                <inertia ixx="1.8792911368909E-05"  ixy="3.31256392204584E-10" ixz="-1.14082001662767E-08"
+                        iyy="3.11510738759073E-05" iyz="-3.60499245082192E-10"
+                        izz="1.88266886146847E-05" />
+            </inertial>
             <visual>
                 <origin rpy="-1.57 0 0" xyz="0 0 0" />

Commit message: control library added

File: urdf/my_robot_gazebo.xacro (robot description, xacro)
@@ -53,5 +53,5 @@
             <robot_param>robot_description</robot_param>
             <robot_param_node>robot_state_publisher</robot_param_node>
-            <parameters></parameters>
+            <parameters>$(find my_robot_controller)/config/my_robot_controller.yaml</parameters>
         </plugin>
     </gazebo>

File: urdf/my_robot_ros2_control.xacro (robot description, xacro)
@@ -1,28 +1,28 @@
 <?xml version ="1.0"?>
 <robot xmlns:xacro="http://www.ros.org/wiki/xacro" name="my_robot">
-<ros2_control type="system" name="RobotSystem">
-    <hardware>
-        <plugin>gazebo_ros2_control/GazeboSystem</plugin>
-    </hardware>
-</ros2_control>
-<joint name="wheel_right_joint" >
-    <command_interface name="velocity">
-        <param name="min">-1</param>
-        <param name="max">1</param>
-    </command_interface>
-    <!--this is the command which send to the motor (in simulator)
-    and have limits min = -1 rad/sec max = 1 rad/ sec-->
-    <state_interface name="position"/>
-    <state_interface name="velocity"/>
-</joint>
-<joint name="wheel_left_joint" >
-    <command_interface name="velocity">
-        <param name="min">-1</param>
-        <param name="max">1</param>
-    </command_interface>
-    <!--this is the command which send to the motor (in simulator)
-    and have limits min = -1 rad/sec max = 1 rad/ sec-->
-    <state_interface name="position"/>
-    <state_interface name="velocity"/>
-</joint>
+    <ros2_control type="system" name="RobotSystem">
+        <hardware>
+            <plugin>gazebo_ros2_control/GazeboSystem</plugin>
+        </hardware>
+        <joint name="base_wheel_left_joint" >
+            <command_interface name="velocity">
+                <param name="min">-1</param>
+                <param name="max">1</param>
+            </command_interface>
+            <!--this is the command which send to the motor (in simulator)
+            and have limits min = -1 rad/sec max = 1 rad/ sec-->
+            <state_interface name="position"/>
+            <state_interface name="velocity"/>
+        </joint>
+        <joint name="base_wheel_right_joint" >
+            <command_interface name="velocity">
+                <param name="min">-1</param>
+                <param name="max">1</param>
+            </command_interface>
+            <!--this is the command which send to the motor (in simulator)
+            and have limits min = -1 rad/sec max = 1 rad/ sec-->
+            <state_interface name="position"/>
+            <state_interface name="velocity"/>
+        </joint>
+    </ros2_control>
 </robot>

File: urdf/robot_urdf.xacro (robot description, xacro)
@@ -2,5 +2,5 @@
 <robot xmlns:xacro="http://www.ros.org/wiki/xacro" name="my_robot">
     <xacro:include filename="$(find my_robot_description)/urdf/my_robot_gazebo.xacro"/>
-<xacro:include filename="$(find my_robot_description)/urdf/urdf/urdf/my_robot_ros2_control.xacro"/>
+    <xacro:include filename="$(find my_robot_description)/urdf/my_robot_ros2_control.xacro"/>
     <link name="base_fooprint"/>
              <!-- footprint usualy the lower part of the robot touched to the ground at point 0 0 0 -->
@@ -126,4 +126,5 @@
         <origin rpy="0 0 0" xyz="0 -0.07 0" />
         <axis xyz="0.0 1.0 0.0"/>
+         <limit effort="5.0" velocity="10.0"/>
     </joint>
  <link name="left_wheel_link">
@@ -157,4 +158,5 @@
         <origin rpy="0 0 0" xyz="0 0.07 0" />
         <axis xyz="0.0 1.0 0.0"/>
+        <limit effort="5.0" velocity="10.0"/>
     </joint>
 </robot>
