Commit message: last uadate 4/3

File: install/my_robot_description/share/my_robot_description/urdf/robot_urdf.xacro (robot description, xacro)
@@ -1,7 +1,16 @@
 <?xml version ="1.0"?>
-<robot xmlns:zacro="http://www.ros.org/wiki/xacro" name="my_robot">
+<robot xmlns:xacro="http://www.ros.org/wiki/xacro" name="my_robot">
+    <xacro:include filename="$(find my_robot_description)/urdf/my_robot_gazebo.xacro"/>
+    <xacro:include filename="$(find my_robot_description)/urdf/my_robot_ros2_control.xacro"/>
     <link name="base_fooprint"/>
              <!-- footprint usualy the lower part of the robot touched to the ground at point 0 0 0 -->
     <link name="base_link">
+        <inertial>
+            <origin xyz="0 0 0.04" rpy="0.0 0.25 0.3" />
+            <mass value="8.2573504e-01"/>
+            <inertia ixx="2.2124416e-02" ixy="-1.2294101e-04" ixz="3.4938785e-04"
+                    iyy="2.1193702e-02" iyz="-5.0120904e-05"
+                    izz="2.0064271e-02" />
+        </inertial>
         <visual>
             <origin rpy="0 0 0" xyz="0 0 0" />
@@ -11,6 +20,13 @@
                </geometry>
                <material name="blue">
-                    <color rgba="0.0 0.0 1.0 1.0"/> <!-- RGB and Alpha values (1.0 = fully opaque) -->
+                    <color rgba="0.0 0.0 1.0 1.0"/>
+                    <!-- RGB and Alpha values (1.0 = fully opaque) -->
                </material>
+               <collision>
+                    <origin rpy="0 0 0" xyz="0 0 0" />
+                    <geometry>
+                        <mesh filename="package://my_robot_description/meshes/base_link.STL" />
+                    </geometry>
+                </collision>
         </visual>
     </link>
@@ -23,4 +39,11 @@
     </joint>
     <link name="caster_wheel_front">
+            <inertial>
+            <origin xyz="3.89968128948481E-07 2.40073004698083E-07 0.00219173397061506" rpy="0 0 0" />
+            <mass value="1.44379265037903E-06" />
+            <inertia ixx="7.23075276010246E-11" ixy="-6.10956883467859E-16" ixz="2.22849693525031E-15"
+                    iyy="3.8713793085917E-11"  iyz="2.93909858781952E-15"
+                    izz="1.00967486676306E-10" />
+            </inertial>
             <visual>
                 <origin rpy="0 0 0" xyz="0 0 0" />
@@ -32,4 +55,10 @@
                 </material>
             </visual>
+            <collision>
+                <origin xyz="0.0 0.0 0.0" rpy="0.0 0.0 0.0"/>
+                <geometry>
+                     <sphere radius="0.005"/>
+                </geometry>
+            </collision>
     </link>
     <joint name="base_caster_wheel_front_joint" type="fixed">
@@ -39,4 +68,11 @@
     </joint>
    <link name="caster_wheel_rear">
+            <inertial>
+            <origin xyz="3.8996812895542E-07 2.40073004698083E-07 0.00219173397061509" rpy="0 0 0" />
+            <mass value="1.44379265037902E-06" />
+            <inertia ixx="7.23075276010246E-11" ixy="-6.10956872363424E-16" ixz="2.22849693527207E-15"
+                    iyy="3.87137930859167E-11" iyz="2.939098587861E-15"
+                    izz="1.00967486676306E-10" />
+            </inertial>
             <visual>
                 <origin rpy="0 0 0" xyz="0 0 0" />
@@ -48,4 +84,10 @@
                 </material>
             </visual>
+            <collision>
+                <origin xyz="0.0 0.0 0.0" rpy="0.0 0.0 0.0"/>
+                <geometry>
+                        <sphere radius="0.005"/>
+                </geometry>
+            </collision>
     </link>
     <joint name="base_caster_wheel_rear_joint" type="fixed">
@@ -55,4 +97,11 @@
     </joint>
     <link name="right_wheel_link">
+            <inertial>
+            <origin xyz="0 -0.014 0" rpy="0 0 0" />
+            <mass value="0.0530086090966721" />
+            <inertia ixx="1.88176298336665E-05" ixy="-4.8444933029987E-10" ixz="1.88163708851143E-08"
+                    iyy="3.11510738647764E-05" iyz="-6.93560663069607E-11"
+                    izz="1.8801969558182E-05" />
+            </inertial>
             <visual>
                 <origin rpy="1.57 0 0" xyz="0 0 0" />
@@ -64,4 +113,11 @@
                 </material>
             </visual>
+            <collision>
+              <origin xyz="0 -0.015 0" rpy="1.57 0 0" />
+                <!-- this origin of the geometry with respect to the link it self-->
+              <geometry>
+                <sphere radius="0.033"/>
+              </geometry>
+            </collision>
     </link>
     <joint name="base_wheel_right_joint" type="continuous">
@@ -70,6 +126,14 @@
         <origin rpy="0 0 0" xyz="0 -0.07 0" />
         <axis xyz="0.0 1.0 0.0"/>
+         <limit effort="5.0" velocity="10.0"/>
     </joint>
  <link name="left_wheel_link">
+           <inertial>
+                <origin xyz="0 0.014 0" rpy="0 0 0" />
+                <mass value="0.0530086043217644" />
+                <inertia ixx="1.8792911368909E-05"  ixy="3.31256392204584E-10" ixz="-1.14082001662767E-08"
+                        iyy="3.11510738759073E-05" iyz="-3.60499245082192E-10"
+                        izz="1.88266886146847E-05" />
+            </inertial>
             <visual>
                 <origin rpy="-1.57 0 0" xyz="0 0 0" />
@@ -81,4 +145,11 @@
                 </material>
             </visual>
+            <collision>
+              <origin xyz="0 0.015 0" rpy="1.57 0 0" />
+                <!-- this origin of the geometry with respect to the link it self-->
+              <geometry>
+                <sphere radius="0.033"/>
+              </geometry>
+            </collision>
     </link>
     <joint name="base_wheel_left_joint" type="continuous">
@@ -87,4 +158,5 @@
         <origin rpy="0 0 0" xyz="0 0.07 0" />
         <axis xyz="0.0 1.0 0.0"/>
+        <limit effort="5.0" velocity="10.0"/>
     </joint>
 </robot>
